File: ncl30105-48V-100W/controller.brd (EAGLE design)
At the start: 50 x 20 mm, 20 parts, among them IC1 NCL30105DR2G, Q1 BCX70SMD

Commit message: Finish rev1.0 changes
Parts:
- removed U$1: N_MOSFET_TO252, power-mosfet:TO252
- added C8: 1uF, rcl:C1210
- added D3: (no value), diode:SMBJ
- added R4: fuse 10A, rcl:R1206
- added T1: N_MOSFET_TO252, power-mosfet:TO252
- C1: device rcl:C1206 -> rcl:C0805
- R3: value 24K9 -> 100K; device rcl:R0603 -> rcl:R1206
- R5: value 0R02 -> NP
- R6: value NP -> 0R02
- moved IN 67.5 mm to (5.00, 4.20)
- moved OUT 49.3 mm to (49.0, 4.20), turned to 180 degrees
- moved R5 36.0 mm to (27.8, 12.4), turned to 270 degrees
- moved IC1 34.1 mm to (20.2, 17.2)
- moved R2 34.1 mm to (24.6, 12.4), turned to 270 degrees
- moved C7 32.7 mm to (11.6, 19.4), turned to 90 degrees
- moved R1 30.9 mm to (16.6, 15.0), turned to 270 degrees
- moved R6 28.4 mm to (31.8, 12.8), turned to 180 degrees
- moved C5 28.3 mm to (27.0, 7.60), turned to 90 degrees
- moved C1 27.4 mm to (9.60, 19.4), turned to 90 degrees
- moved C6 27.2 mm to (20.6, 7.00), turned to 270 degrees
- moved C2 24.9 mm to (16.6, 19.6), turned to 90 degrees
- moved Q1 22.0 mm to (11.6, 14.6), turned to 180 degrees
- moved C4 18.4 mm to (23.8, 7.60), turned to 90 degrees
- moved R3 13.5 mm to (14.6, 14.4), turned to 270 degrees
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Connections:
- new net N$10: IN.1_1, IN.1_2, R4.1
- net GND: now also D3.A, R6.1; no longer R5.1
- net N$1: now also T1.1; no longer U$1.1
- net N$3: now also R5.1, T1.3; no longer R6.1, U$1.3
- net N$5: now also T1.4; no longer U$1.4
- net N$7: now also C8.2
- net VIN: now also C8.1, D3.C, R4.2; no longer IN.1_1, IN.1_2
Routing:
- net VIN: track 0.00 -> 19.9 mm
- net N$8: track 0.00 -> 9.18 mm, vias 0 -> 2
- net N$3: track 0.00 -> 8.39 mm
- net N$4: track 0.00 -> 6.83 mm
- net N$2: track 0.00 -> 4.70 mm
- net N$6: track 0.00 -> 1.88 mm
- added copper zone on layer 1, net GND
- added copper zone on layer 1, net N$1
- added copper zone on layer 1, net N$10
- added copper zone on layer 1, net N$5
- added copper zone on layer 1, net N$7
- added copper zone on layer 1, net N$8
- added copper zone on layer 1, net N$9
- added copper zone on layer 1, net VIN
Other:
- board size 50 x 20 mm -> 46 x 22 mm
