File: ncl30105-48V-100W/controller.sch (EAGLE design)
At the start: 20 parts, among them IC1 NCL30105DR2G, Q1 BCX70SMD

Commit message: Finish rev1.0 changes
Parts:
- added C8: 1uF, rcl:C-EUC1210
- added D3: (no value), diode:SUPPRESSOR-SMBJ
- added R4: fuse 10A, rcl:R-EU_R1206
- C1: device rcl:C-EUC1206 -> rcl:C-EUC0805
- R3: value 24K9 -> 100K; device rcl:R-EU_R0603 -> rcl:R-EU_R1206
- R5: value 0R02 -> NP
- R6: value NP -> 0R02
- renumbered U$1 to T1
Connections:
- new net N$10: IN.1, R4.1
- net GND: now also D3.A, R6.1; no longer R5.1
- net N$3: now also R5.1; no longer R6.1
- net N$7: now also C8.2
- net VIN: now also C8.1, D3.C, R4.2; no longer IN.1
Other:
- moved on the sheet: IN, OUT, R2, R5, R6
